Commit message: spring version

File: resources/robots/mini_cheetah/urdf/spring_mini_cheetah.urdf (robot description, URDF)
Before this commit: robot mini_cheetah, 15 links, 14 joints
Links:
- added link FL_foot, mass 0.0; collision sphere radius=0.0175; visual sphere radius=0.0175
- added link FR_foot, mass 0.0; collision sphere radius=0.0175; visual sphere radius=0.0175
- added link RL_foot, mass 0.0; collision sphere radius=0.0175; visual sphere radius=0.0175
- added link RR_foot, mass 0.0; collision sphere radius=0.0175; visual sphere radius=0.0175
Joints:
- added joint attach: type prismatic, parent FR_calf, child FR_foot, origin xyz=0.0 0.0 -0.21 rpy=0 0 0, axis 0 0 -1, limit lower=-0.1 upper=0.1
- added joint attach2: type prismatic, parent FL_calf, child FL_foot, origin xyz=0.0 0.0 -0.21 rpy=0 0 0, axis 0 0 -1, limit lower=-0.1 upper=0.1
- added joint attach3: type prismatic, parent RR_calf, child RR_foot, origin xyz=0.0 0.0 -0.21 rpy=0 0 0, axis 0 0 -1, limit lower=-0.1 upper=0.1
- added joint attach4: type prismatic, parent RL_calf, child RL_foot, origin xyz=0.0 0.0 -0.21 rpy=0 0 0, axis 0 0 -1, limit lower=-0.1 upper=0.1
